File: 3inaudiomixer.kicad_pcb (KiCad board)
At the start: 2 copper layers, 64 x 72 mm, 50 parts, among them J1 AudioJack3, J2 AudioJack3, J3 AudioJack3, J4 AudioJack3, J5 Conn_01x03_Female, U1 LF353D, U2 LF353D, U3 L78L05_SOT89, U4 L79L05_SOT89

Commit message: changed repo pic
Parts:
- C1, C2, C3, C4, C5, C6: value CP -> 0.1uF
- C10, C7, C8, C9: value C -> 100nF
- C11, C12: value CP -> 10uF
- C13, C14: value CP -> 220uF
- R1, R10, R11, R12, R14, R4, R7: value R -> 100k
- R13: value R -> 22k
- R15: value R -> 20k
- R2, R5, R8: value R -> 10k
- R3, R6, R9: value R -> 1.5M
- RV1, RV2, RV3: value R_POT -> 100k
Changed lines of the file:
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@@
       (drillshape 0)
       (scaleselection 1)
-      (outputdirectory "ensamble/"))
+      (outputdirectory "gerber/"))
   )
   (net 0 "")
@@
       (effects (font (size 1 1) (thickness 0.15)))
     )
-    (fp_text value R (at 0 1.65 90) (layer F.Fab)
+    (fp_text value 20k (at 0 1.65 90) (layer F.Fab)
       (effects (font (size 1 1) (thickness 0.15)))
     )
@@
       (effects (font (size 1 1) (thickness 0.15)))
     )
-    (fp_text value R (at 0 1.65 90) (layer F.Fab)
+    (fp_text value 100k (at 0 1.65 90) (layer F.Fab)
       (effects (font (size 1 1) (thickness 0.15)))
     )
@@
       (effects (font (size 1 1) (thickness 0.15)))
     )
-    (fp_text value R (at 0 1.65 90) (layer F.Fab)
+    (fp_text value 22k (at 0 1.65 90) (layer F.Fab)
       (effects (font (size 1 1) (thickness 0.15)))
     )
@@
       (effects (font (size 1 1) (thickness 0.15)))
     )
-    (fp_text value R (at 0 1.65) (layer F.Fab)
+    (fp_text value 100k (at 0 1.65) (layer F.Fab)
       (effects (font (size 1 1) (thickness 0.15)))
     )
@@
       (effects (font (size 1 1) (thickness 0.15)))
     )
-    (fp_text value R (at 0 1.65) (layer F.Fab)
+    (fp_text value 100k (at 0 1.65) (layer F.Fab)
       (effects (font (size 1 1) (thickness 0.15)))
     )
@@
       (effects (font (size 1 1) (thickness 0.15)))
     )
-    (fp_text value R (at 0 1.65) (layer F.Fab)
+    (fp_text value 100k (at 0 1.65) (layer F.Fab)
       (effects (font (size 1 1) (thickness 0.15)))
     )
@@
       (effects (font (size 1 1) (thickness 0.15)))
     )
-    (fp_text value R (at 0 1.65 90) (layer F.Fab)
+    (fp_text value 1.5M (at 0 1.65 90) (layer F.Fab)
       (effects (font (size 1 1) (thickness 0.15)))
     )
@@
       (effects (font (size 1 1) (thickness 0.15)))
     )
-    (fp_text value R (at 0 1.65 90) (layer F.Fab)
+    (fp_text value 10k (at 0 1.65 90) (layer F.Fab)
       (effects (font (size 1 1) (thickness 0.15)))
     )
@@
       (effects (font (size 1 1) (thickness 0.15)))
     )
-    (fp_text value R (at 0 1.65 90) (layer F.Fab)
+    (fp_text value 100k (at 0 1.65 90) (layer F.Fab)
       (effects (font (size 1 1) (thickness 0.15)))
     )
@@
       (effects (font (size 1 1) (thickness 0.15)))
     )
-    (fp_text value R (at 0 1.65 90) (layer F.Fab)
+    (fp_text value 1.5M (at 0 1.65 90) (layer F.Fab)
       (effects (font (size 1 1) (thickness 0.15)))
     )
@@
       (effects (font (size 1 1) (thickness 0.15)))
     )
-    (fp_text value R (at 0 1.65 90) (layer F.Fab)
+    (fp_text value 10k (at 0 1.65 90) (layer F.Fab)
       (effects (font (size 1 1) (thickness 0.15)))
     )
@@
       (effects (font (size 1 1) (thickness 0.15)))
     )
-    (fp_text value R (at 0 1.65 90) (layer F.Fab)
+    (fp_text value 100k (at 0 1.65 90) (layer F.Fab)
       (effects (font (size 1 1) (thickness 0.15)))
     )
@@
       (effects (font (size 1 1) (thickness 0.15)))
     )
-    (fp_text value R (at 0 1.65 90) (layer F.Fab)
+    (fp_text value 1.5M (at 0 1.65 90) (layer F.Fab)
       (effects (font (size 1 1) (thickness 0.15)))
     )
@@
       (effects (font (size 1 1) (thickness 0.15)))
     )
-    (fp_text value R (at 0 1.65 90) (layer F.Fab)
+    (fp_text value 10k (at 0 1.65 90) (layer F.Fab)
       (effects (font (size 1 1) (thickness 0.15)))
     )
@@
       (effects (font (size 1 1) (thickness 0.15)))
     )
-    (fp_text value R (at 0 1.65 90) (layer F.Fab)
+    (fp_text value 100k (at 0 1.65 90) (layer F.Fab)
       (effects (font (size 1 1) (thickness 0.15)))
     )
@@
       (effects (font (size 1 1) (thickness 0.15)))
     )
-    (fp_text value CP (at 0 4.35 90) (layer F.Fab)
+    (fp_text value 220uF (at 0 4.35 90) (layer F.Fab)
       (effects (font (size 1 1) (thickness 0.15)))
     )
@@
       (effects (font (size 1 1) (thickness 0.15)))
     )
-    (fp_text value CP (at 0 4.35 90) (layer F.Fab)
+    (fp_text value 220uF (at 0 4.35 90) (layer F.Fab)
       (effects (font (size 1 1) (thickness 0.15)))
     )
@@
       (effects (font (size 1 1) (thickness 0.15)))
     )
-    (fp_text value CP (at 0 1.82 90) (layer F.Fab)
+    (fp_text value 10uF (at 0 1.82 90) (layer F.Fab)
       (effects (font (size 1 1) (thickness 0.15)))
     )
@@
       (effects (font (size 1 1) (thickness 0.15)))
     )
-    (fp_text value CP (at 0 1.82 90) (layer F.Fab)
+    (fp_text value 10uF (at 0 1.82 90) (layer F.Fab)
       (effects (font (size 1 1) (thickness 0.15)))
     )
@@
       (effects (font (size 1 1) (thickness 0.15)))
     )
-    (fp_text value C (at 0 1.65 90) (layer F.Fab)
+    (fp_text value 100nF (at 0 1.65 90) (layer F.Fab)
       (effects (font (size 1 1) (thickness 0.15)))
     )
@@
       (effects (font (size 1 1) (thickness 0.15)))
     )
-    (fp_text value C (at 0 1.65 90) (layer F.Fab)
+    (fp_text value 100nF (at 0 1.65 90) (layer F.Fab)
       (effects (font (size 1 1) (thickness 0.15)))
     )
@@
       (effects (font (size 1 1) (thickness 0.15)))
     )
-    (fp_text value C (at 0 1.65 90) (layer F.Fab)
+    (fp_text value 100nF (at 0 1.65 90) (layer F.Fab)
       (effects (font (size 1 1) (thickness 0.15)))
     )
@@
       (effects (font (size 1 1) (thickness 0.15)))
     )
-    (fp_text value C (at 0 1.65 90) (layer F.Fab)
+    (fp_text value 100nF (at 0 1.65 90) (layer F.Fab)
       (effects (font (size 1 1) (thickness 0.15)))
     )
@@
       (effects (font (size 1 1) (thickness 0.15)))
     )
-    (fp_text value CP (at 0 1.65 90) (layer F.Fab)
+    (fp_text value 0.1uF (at 0 1.65 90) (layer F.Fab)
       (effects (font (size 1 1) (thickness 0.15)))
     )
@@
       (effects (font (size 1 1) (thickness 0.15)))
     )
-    (fp_text value CP (at 0 1.65 90) (layer F.Fab)
+    (fp_text value 0.1uF (at 0 1.65 90) (layer F.Fab)
       (effects (font (size 1 1) (thickness 0.15)))
     )
@@
       (effects (font (size 1 1) (thickness 0.15)))
     )
-    (fp_text value CP (at 0 1.65 90) (layer F.Fab)
+    (fp_text value 0.1uF (at 0 1.65 90) (layer F.Fab)
       (effects (font (size 1 1) (thickness 0.15)))
     )
@@
       (effects (font (size 1 1) (thickness 0.15)))
     )
-    (fp_text value CP (at 0 1.65 90) (layer F.Fab)
+    (fp_text value 0.1uF (at 0 1.65 90) (layer F.Fab)
       (effects (font (size 1 1) (thickness 0.15)))
     )
@@
       (effects (font (size 1 1) (thickness 0.15)))
     )
-    (fp_text value CP (at 0 1.65 90) (layer F.Fab)
+    (fp_text value 0.1uF (at 0 1.65 90) (layer F.Fab)
       (effects (font (size 1 1) (thickness 0.15)))
     )
@@
       (effects (font (size 1 1) (thickness 0.15)))
     )
-    (fp_text value CP (at 0 1.65 90) (layer F.Fab)
+    (fp_text value 0.1uF (at 0 1.65 90) (layer F.Fab)
       (effects (font (size 1 1) (thickness 0.15)))
     )
@@
       (effects (font (size 1 1) (thickness 0.15)))
     )
-    (fp_text value R_POT (at 0 4.7) (layer F.Fab)
+    (fp_text value 100k (at 0 4.7) (layer F.Fab)
       (effects (font (size 1 1) (thickness 0.15)))
     )
@@
       (effects (font (size 1 1) (thickness 0.15)))
     )
-    (fp_text value R_POT (at 0 4.7) (layer F.Fab)
+    (fp_text value 100k (at 0 4.7) (layer F.Fab)
       (effects (font (size 1 1) (thickness 0.15)))
     )
@@
       (effects (font (size 1 1) (thickness 0.15)))
     )
-    (fp_text value R_POT (at 0 4.7) (layer F.Fab)
-      (effects (font (size 1 1) (thickness 0.15)))
-    )
+    (fp_text value 100k (at 0 4.7) (layer F.Fab)
+      (effects (font (size 1 1) (thickness 0.15)))
+    )

Commit message: capacitor footprint fix
Parts:
- C11, C12: footprint Capacitor_SMD:C_1206_3216Metric_Pad1.42x1.75mm_HandSolder -> Capacitor_Tantalum_SMD:CP_EIA-3216-18_Kemet-A_Pad1.58x1.35mm_HandSolder
- moved C12 0.08 mm to (140.1, 99.1)
Changed lines of the file:
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@@
     (add_net "Net-(R7-Pad2)")
+  )
+  (module Capacitor_Tantalum_SMD:CP_EIA-3216-18_Kemet-A_Pad1.58x1.35mm_HandSolder (layer F.Cu)
+    (at 140.081 99.06 270)
+    (descr "Tantalum Capacitor SMD Kemet-A (3216-18 Metric), IPC_7351 nominal, (Body size from: http://www.kemet.com/Lists/ProductCatalog/Attachments/253/KEM_TC101_STD.pdf), generated with kicad-footprint-generator")
+    (tags "capacitor tantalum")
+    (attr smd)
+    (fp_text reference C12 (at 0 -1.75 90) (layer F.SilkS)
+      (effects (font (size 1 1) (thickness 0.15)))
+    )
+    (fp_text value 10uF (at 0 1.75 90) (layer F.Fab)
+      (effects (font (size 1 1) (thickness 0.15)))
+    )
+    (fp_text user %R (at 0 0 90) (layer F.Fab)
+      (effects (font (size 0.8 0.8) (thickness 0.12)))
+    )
+    (fp_line (start 2.48 1.05) (end -2.48 1.05) (layer F.CrtYd) (width 0.05))
+    (fp_line (start 2.48 -1.05) (end 2.48 1.05) (layer F.CrtYd) (width 0.05))
+    (fp_line (start -2.48 -1.05) (end 2.48 -1.05) (layer F.CrtYd) (width 0.05))
+    (fp_line (start -2.48 1.05) (end -2.48 -1.05) (layer F.CrtYd) (width 0.05))
+    (fp_line (start -2.485 0.935) (end 1.6 0.935) (layer F.SilkS) (width 0.12))
+    (fp_line (start -2.485 -0.935) (end -2.485 0.935) (layer F.SilkS) (width 0.12))
+    (fp_line (start 1.6 -0.935) (end -2.485 -0.935) (layer F.SilkS) (width 0.12))
+    (fp_line (start 1.6 0.8) (end 1.6 -0.8) (layer F.Fab) (width 0.1))
+    (fp_line (start -1.6 0.8) (end 1.6 0.8) (layer F.Fab) (width 0.1))
+    (fp_line (start -1.6 -0.4) (end -1.6 0.8) (layer F.Fab) (width 0.1))
+    (fp_line (start -1.2 -0.8) (end -1.6 -0.4) (layer F.Fab) (width 0.1))
+    (fp_line (start 1.6 -0.8) (end -1.2 -0.8) (layer F.Fab) (width 0.1))
+    (pad 2 smd roundrect (at 1.4375 0 270) (size 1.575 1.35) (layers F.Cu F.Paste F.Mask) (roundrect_rratio 0.185185)
+      (net 13 "Net-(C10-Pad1)"))
+    (pad 1 smd roundrect (at -1.4375 0 270) (size 1.575 1.35) (layers F.Cu F.Paste F.Mask) (roundrect_rratio 0.185185)
+      (net 15 "Net-(C10-Pad2)"))
+    (model ${KISYS3DMOD}/Capacitor_Tantalum_SMD.3dshapes/CP_EIA-3216-18_Kemet-A.wrl
+      (at (xyz 0 0 0))
+      (scale (xyz 1 1 1))
+      (rotate (xyz 0 0 0))
+    )
+  )
+  (module Capacitor_Tantalum_SMD:CP_EIA-3216-18_Kemet-A_Pad1.58x1.35mm_HandSolder (layer F.Cu)
+    (at 139.954 108.712 90)
+    (descr "Tantalum Capacitor SMD Kemet-A (3216-18 Metric), IPC_7351 nominal, (Body size from: http://www.kemet.com/Lists/ProductCatalog/Attachments/253/KEM_TC101_STD.pdf), generated with kicad-footprint-generator")
+    (tags "capacitor tantalum")
+    (attr smd)
+    (fp_text reference C11 (at 0 -1.75 90) (layer F.SilkS)
+      (effects (font (size 1 1) (thickness 0.15)))
+    )
+    (fp_text value 10uF (at 0 1.75 90) (layer F.Fab)
+      (effects (font (size 1 1) (thickness 0.15)))
+    )
+    (fp_text user %R (at 0 0 90) (layer F.Fab)
+      (effects (font (size 0.8 0.8) (thickness 0.12)))
+    )
+    (fp_line (start 2.48 1.05) (end -2.48 1.05) (layer F.CrtYd) (width 0.05))
+    (fp_line (start 2.48 -1.05) (end 2.48 1.05) (layer F.CrtYd) (width 0.05))
+    (fp_line (start -2.48 -1.05) (end 2.48 -1.05) (layer F.CrtYd) (width 0.05))
+    (fp_line (start -2.48 1.05) (end -2.48 -1.05) (layer F.CrtYd) (width 0.05))
+    (fp_line (start -2.485 0.935) (end 1.6 0.935) (layer F.SilkS) (width 0.12))
+    (fp_line (start -2.485 -0.935) (end -2.485 0.935) (layer F.SilkS) (width 0.12))
+    (fp_line (start 1.6 -0.935) (end -2.485 -0.935) (layer F.SilkS) (width 0.12))
+    (fp_line (start 1.6 0.8) (end 1.6 -0.8) (layer F.Fab) (width 0.1))
+    (fp_line (start -1.6 0.8) (end 1.6 0.8) (layer F.Fab) (width 0.1))
+    (fp_line (start -1.6 -0.4) (end -1.6 0.8) (layer F.Fab) (width 0.1))
+    (fp_line (start -1.2 -0.8) (end -1.6 -0.4) (layer F.Fab) (width 0.1))
+    (fp_line (start 1.6 -0.8) (end -1.2 -0.8) (layer F.Fab) (width 0.1))
+    (pad 2 smd roundrect (at 1.4375 0 90) (size 1.575 1.35) (layers F.Cu F.Paste F.Mask) (roundrect_rratio 0.185185)
+      (net 13 "Net-(C10-Pad1)"))
+    (pad 1 smd roundrect (at -1.4375 0 90) (size 1.575 1.35) (layers F.Cu F.Paste F.Mask) (roundrect_rratio 0.185185)
+      (net 14 "Net-(C11-Pad1)"))
+    (model ${KISYS3DMOD}/Capacitor_Tantalum_SMD.3dshapes/CP_EIA-3216-18_Kemet-A.wrl
+      (at (xyz 0 0 0))
+      (scale (xyz 1 1 1))
+      (rotate (xyz 0 0 0))
+    )
   )
   (module Logos_Caty_Kanal:CATY-KANAL-Logo_18x8mm_SilkScreen (layer F.Cu)
@@
       (at (xyz 0 0 0))
       (scale (xyz 1 1 1))
-      (rotate (xyz 0 0 0))
-    )
-  )
-  (module Capacitor_SMD:C_1206_3216Metric_Pad1.42x1.75mm_HandSolder (layer F.Cu)
-    (at 140 99.06 270)
-    (descr "Capacitor SMD 1206 (3216 Metric), square (rectangular) end terminal, IPC_7351 nominal with elongated pad for handsoldering. (Body size source: http://www.tortai-tech.com/upload/download/2011102023233369053.pdf), generated with kicad-footprint-generator")
-    (tags "capacitor handsolder")
-    (attr smd)
-    (fp_text reference C12 (at 0.127 -2.113 90) (layer F.SilkS)
-      (effects (font (size 1 1) (thickness 0.15)))
-    )
-    (fp_text value 10uF (at 0 1.82 90) (layer F.Fab)
-      (effects (font (size 1 1) (thickness 0.15)))
-    )
-    (fp_text user %R (at 0 0 90) (layer F.Fab)
-      (effects (font (size 0.8 0.8) (thickness 0.12)))
-    )
-    (fp_line (start 2.45 1.12) (end -2.45 1.12) (layer F.CrtYd) (width 0.05))
-    (fp_line (start 2.45 -1.12) (end 2.45 1.12) (layer F.CrtYd) (width 0.05))
-    (fp_line (start -2.45 -1.12) (end 2.45 -1.12) (layer F.CrtYd) (width 0.05))
-    (fp_line (start -2.45 1.12) (end -2.45 -1.12) (layer F.CrtYd) (width 0.05))
-    (fp_line (start -0.602064 0.91) (end 0.602064 0.91) (layer F.SilkS) (width 0.12))
-    (fp_line (start -0.602064 -0.91) (end 0.602064 -0.91) (layer F.SilkS) (width 0.12))
-    (fp_line (start 1.6 0.8) (end -1.6 0.8) (layer F.Fab) (width 0.1))
-    (fp_line (start 1.6 -0.8) (end 1.6 0.8) (layer F.Fab) (width 0.1))
-    (fp_line (start -1.6 -0.8) (end 1.6 -0.8) (layer F.Fab) (width 0.1))
-    (fp_line (start -1.6 0.8) (end -1.6 -0.8) (layer F.Fab) (width 0.1))
-    (pad 2 smd roundrect (at 1.4875 0 270) (size 1.425 1.75) (layers F.Cu F.Paste F.Mask) (roundrect_rratio 0.175439)
-      (net 13 "Net-(C10-Pad1)"))
-    (pad 1 smd roundrect (at -1.4875 0 270) (size 1.425 1.75) (layers F.Cu F.Paste F.Mask) (roundrect_rratio 0.175439)
-      (net 15 "Net-(C10-Pad2)"))
-    (model ${KISYS3DMOD}/Capacitor_SMD.3dshapes/C_1206_3216Metric.wrl
-      (at (xyz 0 0 0))
-      (scale (xyz 1 1 1))
-      (rotate (xyz 0 0 0))
-    )
-  )
-  (module Capacitor_SMD:C_1206_3216Metric_Pad1.42x1.75mm_HandSolder (layer F.Cu)
-    (at 140 108.712 90)
-    (descr "Capacitor SMD 1206 (3216 Metric), square (rectangular) end terminal, IPC_7351 nominal with elongated pad for handsoldering. (Body size source: http://www.tortai-tech.com/upload/download/2011102023233369053.pdf), generated with kicad-footprint-generator")
-    (tags "capacitor handsolder")
-    (attr smd)
-    (fp_text reference C11 (at 0 2.113 90) (layer F.SilkS)
-      (effects (font (size 1 1) (thickness 0.15)))
-    )
-    (fp_text value 10uF (at 0 1.82 90) (layer F.Fab)
-      (effects (font (size 1 1) (thickness 0.15)))
-    )
-    (fp_text user %R (at 0 0 90) (layer F.Fab)
-      (effects (font (size 0.8 0.8) (thickness 0.12)))
-    )
-    (fp_line (start 2.45 1.12) (end -2.45 1.12) (layer F.CrtYd) (width 0.05))
-    (fp_line (start 2.45 -1.12) (end 2.45 1.12) (layer F.CrtYd) (width 0.05))
-    (fp_line (start -2.45 -1.12) (end 2.45 -1.12) (layer F.CrtYd) (width 0.05))
-    (fp_line (start -2.45 1.12) (end -2.45 -1.12) (layer F.CrtYd) (width 0.05))
-    (fp_line (start -0.602064 0.91) (end 0.602064 0.91) (layer F.SilkS) (width 0.12))
-    (fp_line (start -0.602064 -0.91) (end 0.602064 -0.91) (layer F.SilkS) (width 0.12))
-    (fp_line (start 1.6 0.8) (end -1.6 0.8) (layer F.Fab) (width 0.1))
-    (fp_line (start 1.6 -0.8) (end 1.6 0.8) (layer F.Fab) (width 0.1))
-    (fp_line (start -1.6 -0.8) (end 1.6 -0.8) (layer F.Fab) (width 0.1))
-    (fp_line (start -1.6 0.8) (end -1.6 -0.8) (layer F.Fab) (width 0.1))
-    (pad 2 smd roundrect (at 1.4875 0 90) (size 1.425 1.75) (layers F.Cu F.Paste F.Mask) (roundrect_rratio 0.175439)
-      (net 13 "Net-(C10-Pad1)"))
-    (pad 1 smd roundrect (at -1.4875 0 90) (size 1.425 1.75) (layers F.Cu F.Paste F.Mask) (roundrect_rratio 0.175439)
-      (net 14 "Net-(C11-Pad1)"))
-    (model ${KISYS3DMOD}/Capacitor_SMD.3dshapes/C_1206_3216Metric.wrl
-      (at (xyz 0 0 0))
-      (scale (xyz 1 1 1))

Commit message: removed voltage regulators
Parts:
- removed U3: L78L05_SOT89, Package_TO_SOT_SMD:SOT-89-3
- removed U4: L79L05_SOT89, Package_TO_SOT_SMD:SOT-89-3
Connections:
- C13 pad 1: Net-(C13-Pad1) -> Net-(C11-Pad1)
- C14 pad 1: Net-(C14-Pad1) -> Net-(C10-Pad2)
- J5 pad 1: Net-(C14-Pad1) -> Net-(C10-Pad2)
- J5 pad 3: Net-(C13-Pad1) -> Net-(C11-Pad1)
Routing:
- net Net-(C11-Pad1): track 85.7 -> 108.4 mm, vias 6 -> 8
- net Net-(C10-Pad2): track 77.0 -> 98.7 mm
- net Net-(C14-Pad1): track 20.2 -> 0.00 mm
- net Net-(C13-Pad1): track 19.6 -> 0.00 mm
- net Net-(C10-Pad1): track 323.7 -> 320.2 mm
